Commit message: update to noetic

File: urdf/robot.xacro (robot description, xacro)
@@ -3,6 +3,6 @@
  <xacro:include filename="$(find nexus_gelo)/urdf/nexus/nexus_4wd_mecanum.xacro"/>
  <include filename="$(find nexus_gelo)/urdf/sensors/lidar.xacro"/>
- <xacro:laser>
- 	<origin xyz="0 0 0.07" rpy="0 0 0"/>
- </xacro:laser>
+ <!--xacro:laser>
+    <origin xyz="0 0 0.07" rpy="0 0 0" />
+ </xacro:laser-->
 </robot>

File: urdf/sensors/lidar.xacro (robot description, xacro)
@@ -2,10 +2,11 @@
 <robot xmlns:xacro="http://www.ros.org/wiki/xacro" >
     <xacro:include filename="$(find nexus_gelo)/urdf/inercia.xacro"/>
-    <xacro:macro name="laser" params="*origin">
+    <!--xacro:macro name="laser" params="*origin"-->
     <xacro:arg name="robot_name" default="default_robot" />
     <joint name="laser_joint" type="fixed">
         <parent link="base_link"/>
         <child link="laser_frame"/>
-        <xacro:insert_block name="origin" />
+        <!--xacro:insert_block name="origin" /-->
+        <origin xyz="0 0 0.07" rpy="0 0 0" />
     </joint>
     <link name="laser_frame">

Commit message: add imu sensor

File: urdf/robot.xacro (robot description, xacro)
@@ -1,8 +1,6 @@
 <?xml version="1.0"?>
 <robot xmlns:xacro="http://www.ros.org/wiki/xacro" name="juninho" >
- <xacro:include filename="$(find nexus_gelo)/urdf/nexus/nexus_4wd_mecanum.xacro"/>
- <include filename="$(find nexus_gelo)/urdf/sensors/lidar.xacro"/>
- <!--xacro:laser>
-    <origin xyz="0 0 0.07" rpy="0 0 0" />
- </xacro:laser-->
+   <xacro:include filename="$(find nexus_gelo)/urdf/nexus/nexus_4wd_mecanum.xacro"/>
+   <xacro:include filename="$(find nexus_gelo)/urdf/sensors/lidar.xacro"/>
+   <xacro:include filename="$(find nexus_gelo)/urdf/sensors/imu.xacro"/>
 </robot>

File: urdf/sensors/lidar.xacro (robot description, xacro)
@@ -61,4 +61,4 @@
         </sensor>
     </gazebo>
-	</xacro:macro>
+	<!--/xacro:macro-->
 </robot>
